Commit message: Small debugs

File: CPRMover6.urdf (robot description, URDF)
Before this commit: robot CPRMover6, 15 links, 14 joints
Links:
- removed link Body4Back
- added link Body3TopBox; visual box size=0.1 0.07 0.04
- link Body2Oben: geometry visual cylinder length=0.01 radius=0.05
- link Body3: geometry visual cylinder length=0.13 radius=0.05
Joints:
- removed joint A4basetoA4Backfixed
- added joint A3basetoA3TopBoxfixed: type fixed, parent Body3, child Body3TopBox, origin xyz=0 0 0
